File: layout/ArduDisFace.kicad_pcb (KiCad board)
At the start: 2 copper layers, 62 x 56 mm, 55 parts, among them IC1 ATmega328P-AU, IC2 LP2950-5.0_TO252, Q1 16MHz, Q2 BSS138, Q4 BSS138, X1 Power, X2 ISCP, X3 RS232-RPI, X3a1 Prog, X4 LCD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

Commit message: Touch interface with only one ADC input. Usin D3 for direction input
Signed-off-by: Claus Zielke <info@cszielke.de>
Parts:
- removed JP1: D2/A4=En, Jumper:SolderJumper-3_P1.3mm_Bridged12_RoundedPad1.0x1.5mm_NumberLabels
- removed JP4: RW-A2, Jumper:SolderJumper-3_P1.3mm_Bridged12_RoundedPad1.0x1.5mm_NumberLabels
- removed R15: 47, Resistor_SMD:R_0603_1608Metric
- added U1: 4052, Package_SO:SOIC-16_3.9x9.9mm_P1.27mm, B.Cu at (135.8, 95.4)
- added U2: 4052, Package_SO:SOIC-16_3.9x9.9mm_P1.27mm, B.Cu at (149.0, 95.6)
- JP2: value SolderJumper_2_Open -> Vin=5V
- LED1: value grün -> 5V
- LED2: value grün -> D13
- LED3: value grün -> Vin
- R13, R14: value 1K -> 100K
- moved R14 49.4 mm to (108.5, 54.3), turned to 180 degrees
- moved R13 15.2 mm to (137.7, 97.3)
- moved R5 0.51 mm to (158.4, 92.5)
Connections:
- R13 pad 1: /A6 -> /A7
- R14 pad 1: /A7 -> /A6
- X1 pad 3: /D3 -> /A6
- X4 pad 4: /A3 -> /D3
- X4 pad 5: Net-(JP4-Pad2) -> GND
- X4 pad 6: Net-(JP1-Pad2) -> /D2
- X4A1 pad 4: /A3 -> /D3
- X4A1 pad 5: Net-(JP4-Pad2) -> GND
- X4A1 pad 6: Net-(JP1-Pad2) -> /D2
- X4B1 pad 4: /A3 -> /D3
- X4B1 pad 5: Net-(JP4-Pad2) -> GND
- X4B1 pad 6: Net-(JP1-Pad2) -> /D2
- X6 pad 2: /A6 -> Net-(U2-Pad3)
- X6 pad 3: /A7 -> Net-(U1-Pad13)
- X6 pad 4: GND -> Net-(U1-Pad3)
Routing:
- net /A7: track 75.5 -> 125.2 mm, vias 4 -> 10
- net Net-(U1-Pad3): track 0.00 -> 41.6 mm, vias 0 -> 3
- net Net-(U2-Pad3): track 0.00 -> 29.3 mm, vias 0 -> 2
- net Net-(U2-Pad13): track 2.96 -> 28.0 mm, vias 0 -> 2
- net /A2: track 20.5 -> 42.8 mm, vias 0 -> 3
- net Net-(U1-Pad13): track 0.00 -> 20.7 mm, vias 0 -> 1
- net /A4: track 49.4 -> 33.1 mm, vias 5 -> 3
- net VCC: track 225.5 -> 210.4 mm, vias 4 -> 11
- net Net-(JP4-Pad2): track 14.3 -> 0.00 mm
- net GND: track 136.4 -> 150.5 mm, vias 23 -> 24
- net Net-(JP1-Pad2): track 8.63 -> 0.00 mm
- net /D3: track 31.1 -> 39.2 mm, vias 2 -> 4
- net /D2: track 36.8 -> 43.6 mm, vias 4 -> 2
- net /A3: track 40.8 -> 44.3 mm, vias 0 -> 3
- net /D13: track 57.8 -> 60.6 mm
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